File: boards/a1_micro_atx/a1_micro_atx.kicad_pcb (KiCad board)
At the start: 4 copper layers, 243.8 x 204.5 mm, 243 parts, among them J1 Conn_01x01, J10 HDMI_A, J11 SJ1-3535NG-BE, J12 DE9_Plug, J13 Micro_SD_Card, J15 USB_A_Stacked, J16 USB_A_Stacked, J17 USB_A_Stacked, J18 Bus_ISA_8bit, J19 Bus_ISA_8bit, J2 Conn_01x01, J20 Bus_ISA_16bit, J21 Bus_ISA_16bit, J22 Conn_01x01, J23 Conn_01x01, J24 Conn_01x01, J3 Conn_01x01, J4 Conn_01x01, J5 Conn_01x02, J6 Jack-DC, J7 Conn_02x05_Odd_Even, J8 SJ1-3535NG-BE, J9 Conn_01x02, SW2 SW_Push, SW3 SW_Push, SW4 SW_Push, SW5 SW_Push, U1 74LS08, U10 74AHCT245, U11 SST39SF040, U12 A1_POWER, U13 74AHCT245, U14 74AHCT245, U15 74AHCT245, U16 74LS273, U17 74LS273, U18 74LS273, U19 ESPRESSO, U2 74LS86, U20 SIMM-30x2, U21 SIMM-30x2, U22 DISCO, U23 A1_CODEC, U24 MAX232, U25 MIO, U26 DS1307+, U27 KSZ8851-11MLL, U28 A1_USBHUB, U29 L78L33ABZ-AP, U3 74LS00, U30 74AHCT245, U31 74AHCT14, U32 74AHCT139, U33 4075, U34 MC33063AP, U35 L79L05_TO92, U36 MC33063AP, U37 74AHCT245, U38 74HCT153, U4 74LS273, U40 L78L05_TO92, U41 74LS00, U43 ATtiny25-20P, U5 74LS574, U6 74LS139, U7 74LS14, U8 74LS126, U9 74AHCT245, X1 8MHz, X2 CXO_DIP14, X3 24MHz, X4 14.31818MHz, Y1 32768Hz, Y2 25MHz

Commit message: Found some net naming errors. Fixed.
Connections:
- net Net-(J5-Pin_2) renamed /BOOT SELECT
- U5 pad 11: unconnected-(U5-Cp-Pad11) -> /BUF_NREN
