File: boards/a1_micro_atx/a1_micro_atx.kicad_sch (KiCad schematic)
At the start: 76 parts, among them J1 Conn_01x01, J2 Conn_01x01, J22 Conn_01x01, J23 Conn_01x01, J24 Conn_01x01, J3 Conn_01x01, J4 Conn_01x01, J5 Conn_01x02, J6 Jack-DC, SW2 SW_Push, SW3 SW_Push, SW4 SW_Push, SW5 SW_Push, U1 74LS08, U10 74AHCT245, U11 SST39SF040, U12 A1_POWER, U13 74AHCT245, U14 74AHCT245, U15 74AHCT245, U16 74LS273, U17 74LS273, U18 74LS273, U2 74LS86, U3 74LS00, U4 74LS273, U40 L78L05_TO92, U43 ATtiny25-20P, U5 74LS574, U6 74LS139, U7 74LS14, U8 74LS126, U9 74AHCT245, X1 8MHz

Commit message: Found some net naming errors. Fixed.
Connections:
- net BUF_NREN: now also U5.11 (Cp)
- net BOOT SELECT: now reaches J5.2 (Pin_2), RN4.9 (R8), U5.2 (D0)
Other:
- sheet ISA ports: added none; removed ISA_DACK
- note removed: "BOOT SELECT"
- note removed: "BUF_NREN"
