File: boards/a1_micro_atx/memory.kicad_sch (KiCad schematic)
At the start: 4 parts, among them U21 SIMM-30x2

Commit message: Found some net naming errors. Fixed.
Parts:
- renumbered C21 to C51, C22 to C52, C23 to C53
